File: electronics/Spar7_rebuild.brd (EAGLE design)
At the start: 57.1 x 68.2 mm, 42 parts, among them J1 MOLEX-39532-1002, J2 SPAR7_REWIRED_TERM_BLOCK, J3 MOLEX-39532-1002, J4 10118192-0001LF, U1 TPS62172DSGR, U3 ESP32-S3-WROOM-1U-N16R8, U4 CP2102N-A02-GQFN20QFN20_CP210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, U5 CD4511BNSR, U6 ULN2003D1013TR

Commit message: WIP
Parts:
- R10, R11, R12, R13, R14, R9: value 10k 0402 -> (none)
- R16, R17, R18, R19, R20, R21, R22: value 510ohm 1/4W 402 -> (none)
