File: electronics/Spar7_rebuild.sch (EAGLE design)
At the start: 42 parts, among them J1 MOLEX-39532-1002, J2 SPAR7_REWIRED_TERM_BLOCK, J3 MOLEX-39532-1002, J4 10118192-0001LF, U1 TPS62172DSGR, U3 ESP32-S3-WROOM-1U-N16R8, U4 CP2102N-A02-GQFN20QFN20_CP210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, U5 CD4511BNSR, U6 ULN2003D1013TR

Commit message: WIP
Parts:
- R10, R11, R12, R13, R14, R9: value 10k 0402 -> RESISTOR0402
- R16, R17, R18, R19, R20, R21, R22: value 510ohm 1/4W 402 -> RESISTOR0402
Changed lines of the file:
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@@
 </classes>
 <parts>
-<part name="U1" library="TimeExpander2" library_urn="urn:adsk.eagle:library:21801758" deviceset="TPS62173DSGR" device="" package3d_urn="urn:adsk.eagle:package:21801953/3" value="TPS62172DSGR"/>
+<part name="U1" library="TimeExpander2" library_urn="urn:adsk.eagle:library:21801758" deviceset="TPS62173DSGR" device="" package3d_urn="urn:adsk.eagle:package:21801953/4" value="TPS62172DSGR"/>
 <part name="C1" library="TimeExpander2" library_urn="urn:adsk.eagle:library:21801758" deviceset="CAPACITOR" device="0805" package3d_urn="urn:adsk.eagle:package:40605865/1" value="10uF 20V 0805"/>
 <part name="C2" library="TimeExpander2" library_urn="urn:adsk.eagle:library:21801758" deviceset="CAPACITOR" device="1206" package3d_urn="urn:adsk.eagle:package:21801948/2" value="22uF 10V 1206"/>
 <part name="R1" library="TimeExpander2" library_urn="urn:adsk.eagle:library:21801758" deviceset="RESISTOR" device="0402" package3d_urn="urn:adsk.eagle:package:21801914/2" value=""/>
-<part name="L1" library="TimeExpander2" library_urn="urn:adsk.eagle:library:21801758" deviceset="NR3015T2R2M" device="" package3d_urn="urn:adsk.eagle:package:21801952/2"/>
+<part name="L1" library="TimeExpander2" library_urn="urn:adsk.eagle:library:21801758" deviceset="NR3015T2R2M" device="" package3d_urn="urn:adsk.eagle:package:21801952/3"/>
 <part name="GND1" library="TimeExpander2" library_urn="urn:adsk.eagle:library:21801758" deviceset="GND" device=""/>
 <part name="GND2" library="TimeExpander2" library_urn="urn:adsk.eagle:library:21801758" deviceset="GND" device=""/>
@@
 <part name="U3" library="TimeExpander2" library_urn="urn:adsk.eagle:library:21801758" deviceset="ESP32-S3-WROOM-1U-N16R8" device="" package3d_urn="urn:adsk.eagle:package:39030203/1"/>
 <part name="GND30" library="TimeExpander2" library_urn="urn:adsk.eagle:library:21801758" deviceset="GND" device=""/>
-<part name="U4" library="TimeExpander2" library_urn="urn:adsk.eagle:library:21801758" deviceset="CP2102N-A02-GQFN20" device="QFN20_CP2102N_SIL-L" package3d_urn="urn:adsk.eagle:package:39098833/1"/>
+<part name="U4" library="TimeExpander2" library_urn="urn:adsk.eagle:library:21801758" deviceset="CP2102N-A02-GQFN20" device="QFN20_CP2102N_SIL-L" package3d_urn="urn:adsk.eagle:package:39098833/2"/>
 <part name="J4" library="TimeExpander2" library_urn="urn:adsk.eagle:library:21801758" deviceset="USB_RCPT_10118192-0001LF" device="" package3d_urn="urn:adsk.eagle:package:21801967/1" value="10118192-0001LF"/>
 <part name="GND31" library="TimeExpander2" library_urn="urn:adsk.eagle:library:21801758" deviceset="GND" device=""/>
@@
 <part name="DISPLAY" library="TimeExpander2" library_urn="urn:adsk.eagle:library:21801758" deviceset="ELS-1005IDR-SA10-21EWA" device="" package3d_urn="urn:adsk.eagle:package:42753161/1"/>
 <part name="U6" library="EE_copy" deviceset="ULN2003D1013TR" device=""/>
-<part name="R9" library="TimeExpander2" library_urn="urn:adsk.eagle:library:21801758" deviceset="RESISTOR" device="0402" package3d_urn="urn:adsk.eagle:package:21801914/2" value="10k 0402"/>
-<part name="R10" library="TimeExpander2" library_urn="urn:adsk.eagle:library:21801758" deviceset="RESISTOR" device="0402" package3d_urn="urn:adsk.eagle:package:21801914/2" value="10k 0402"/>
-<part name="R11" library="TimeExpander2" library_urn="urn:adsk.eagle:library:21801758" deviceset="RESISTOR" device="0402" package3d_urn="urn:adsk.eagle:package:21801914/2" value="10k 0402"/>
-<part name="R12" library="TimeExpander2" library_urn="urn:adsk.eagle:library:21801758" deviceset="RESISTOR" device="0402" package3d_urn="urn:adsk.eagle:package:21801914/2" value="10k 0402"/>
-<part name="R13" library="TimeExpander2" library_urn="urn:adsk.eagle:library:21801758" deviceset="RESISTOR" device="0402" package3d_urn="urn:adsk.eagle:package:21801914/2" value="10k 0402"/>
-<part name="R14" library="TimeExpander2" library_urn="urn:adsk.eagle:library:21801758" deviceset="RESISTOR" device="0402" package3d_urn="urn:adsk.eagle:package:21801914/2" value="10k 0402"/>
+<part name="R9" library="TimeExpander2" library_urn="urn:adsk.eagle:library:21801758" deviceset="RESISTOR" device="0402" package3d_urn="urn:adsk.eagle:package:21801914/2" value=""/>
+<part name="R10" library="TimeExpander2" library_urn="urn:adsk.eagle:library:21801758" deviceset="RESISTOR" device="0402" package3d_urn="urn:adsk.eagle:package:21801914/2" value=""/>
+<part name="R11" library="TimeExpander2" library_urn="urn:adsk.eagle:library:21801758" deviceset="RESISTOR" device="0402" package3d_urn="urn:adsk.eagle:package:21801914/2" value=""/>
+<part name="R12" library="TimeExpander2" library_urn="urn:adsk.eagle:library:21801758" deviceset="RESISTOR" device="0402" package3d_urn="urn:adsk.eagle:package:21801914/2" value=""/>
+<part name="R13" library="TimeExpander2" library_urn="urn:adsk.eagle:library:21801758" deviceset="RESISTOR" device="0402" package3d_urn="urn:adsk.eagle:package:21801914/2" value=""/>
+<part name="R14" library="TimeExpander2" library_urn="urn:adsk.eagle:library:21801758" deviceset="RESISTOR" device="0402" package3d_urn="urn:adsk.eagle:package:21801914/2" value=""/>
 <part name="USB" library="TimeExpander2" library_urn="urn:adsk.eagle:library:21801758" deviceset="LED" device="150120BS75000" package3d_urn="urn:adsk.eagle:package:40656539/2" value="150120BS75000"/>
 <part name="R4" library="TimeExpander2" library_urn="urn:adsk.eagle:library:21801758" deviceset="RESISTOR" device="0402" package3d_urn="urn:adsk.eagle:package:21801914/2" value=""/>
 <part name="GND9" library="TimeExpander2" library_urn="urn:adsk.eagle:library:21801758" deviceset="GND" device=""/>
-<part name="R16" library="TimeExpander2" library_urn="urn:adsk.eagle:library:21801758" deviceset="RESISTOR" device="0402" package3d_urn="urn:adsk.eagle:package:21801914/2" value="510ohm 1/4W 402"/>
-<part name="R17" library="TimeExpander2" library_urn="urn:adsk.eagle:library:21801758" deviceset="RESISTOR" device="0402" package3d_urn="urn:adsk.eagle:package:21801914/2" value="510ohm 1/4W 402"/>
-<part name="R18" library="TimeExpander2" library_urn="urn:adsk.eagle:library:21801758" deviceset="RESISTOR" device="0402" package3d_urn="urn:adsk.eagle:package:21801914/2" value="510ohm 1/4W 402"/>
-<part name="R19" library="TimeExpander2" library_urn="urn:adsk.eagle:library:21801758" deviceset="RESISTOR" device="0402" package3d_urn="urn:adsk.eagle:package:21801914/2" value="510ohm 1/4W 402"/>
-<part name="R20" library="TimeExpander2" library_urn="urn:adsk.eagle:library:21801758" deviceset="RESISTOR" device="0402" package3d_urn="urn:adsk.eagle:package:21801914/2" value="510ohm 1/4W 402"/>
-<part name="R21" library="TimeExpander2" library_urn="urn:adsk.eagle:library:21801758" deviceset="RESISTOR" device="0402" package3d_urn="urn:adsk.eagle:package:21801914/2" value="510ohm 1/4W 402"/>
-<part name="R22" library="TimeExpander2" library_urn="urn:adsk.eagle:library:21801758" deviceset="RESISTOR" device="0402" package3d_urn="urn:adsk.eagle:package:21801914/2" value="510ohm 1/4W 402"/>
+<part name="R16" library="TimeExpander2" library_urn="urn:adsk.eagle:library:21801758" deviceset="RESISTOR" device="0402" package3d_urn="urn:adsk.eagle:package:21801914/2" value=""/>
+<part name="R17" library="TimeExpander2" library_urn="urn:adsk.eagle:library:21801758" deviceset="RESISTOR" device="0402" package3d_urn="urn:adsk.eagle:package:21801914/2" value=""/>
+<part name="R18" library="TimeExpander2" library_urn="urn:adsk.eagle:library:21801758" deviceset="RESISTOR" device="0402" package3d_urn="urn:adsk.eagle:package:21801914/2" value=""/>
+<part name="R19" library="TimeExpander2" library_urn="urn:adsk.eagle:library:21801758" deviceset="RESISTOR" device="0402" package3d_urn="urn:adsk.eagle:package:21801914/2" value=""/>
+<part name="R20" library="TimeExpander2" library_urn="urn:adsk.eagle:library:21801758" deviceset="RESISTOR" device="0402" package3d_urn="urn:adsk.eagle:package:21801914/2" value=""/>
+<part name="R21" library="TimeExpander2" library_urn="urn:adsk.eagle:library:21801758" deviceset="RESISTOR" device="0402" package3d_urn="urn:adsk.eagle:package:21801914/2" value=""/>
+<part name="R22" library="TimeExpander2" library_urn="urn:adsk.eagle:library:21801758" deviceset="RESISTOR" device="0402" package3d_urn="urn:adsk.eagle:package:21801914/2" value=""/>
 <part name="GND10" library="TimeExpander2" library_urn="urn:adsk.eagle:library:21801758" deviceset="GND" device=""/>
 <part name="GND11" library="TimeExpander2" library_urn="urn:adsk.eagle:library:21801758" deviceset="GND" device=""/>
